File: golmidi.kicad_pcb (KiCad board)
At the start: 2 copper layers, 6.6 x 15.2 mm, 29 parts, among them J1 USB-C, J2 01x02, J3 01x12, J4 01x12, J5 01x05, U1 ATmega32U4, U2 MAX7219, X1 16MHz

Commit message: fixed overlapping traces
Parts:
- removed RV1, RV2: R_POT, Potentiometer_SMD:Potentiometer_ACP_CA6-VSMD_Vertical
- R7: value R -> 9.53k
- moved U2 18.2 mm to (62.5, 73.2)
Connections:
- net Net-(J1-PadA10) renamed no_connect_(J1-PadA10)
- net Net-(J1-PadA11) renamed no_connect_(J1-PadA11)
- net Net-(J1-PadA2) renamed no_connect_(J1-PadA2)
- net Net-(J1-PadA3) renamed no_connect_(J1-PadA3)
- net Net-(J1-PadA8) renamed no_connect_(J1-PadA8)
- net Net-(J1-PadB10) renamed no_connect_(J1-PadB10)
- net Net-(J1-PadB11) renamed no_connect_(J1-PadB11)
- net Net-(J1-PadB2) renamed no_connect_(J1-PadB2)
- net Net-(J1-PadB3) renamed no_connect_(J1-PadB3)
- net Net-(J1-PadB8) renamed no_connect_(J1-PadB8)
- net Net-(U1-Pad26) renamed no_connect_(U1-Pad26)
- net Net-(U1-Pad8) renamed no_connect_(U1-Pad8)
- net Net-(U2-Pad24) renamed no_connect_(U2-Pad24)
- U1 pad 10: Net-(U1-Pad10) -> /PB2
- U1 pad 11: Net-(U1-Pad11) -> /PB3
Other:
- net class Default removed
