File: golmidi.kicad_pcb (KiCad board)
At the start: 2 copper layers, 6.6 x 15.2 mm, 29 parts, among them J1 USB-C, J2 01x02, J3 01x12, J4 01x12, J5 01x05, U1 ATmega32U4, U2 MAX7219, X1 16MHz

Commit message: Started to clean pcb-layout
Parts:
- removed J3, J4: 01x12, pins:Pins12
- removed J5: 01x05, pins:Pins5
- moved D2 124.4 mm to (215.9, 49.5), turned to 180 degrees
- moved U2 101.0 mm to (177.8, 43.2)
- moved R1 58.5 mm to (113.0, 52.1)
- moved C10 45.6 mm to (97.8, 49.5)
- moved C1 43.0 mm to (97.0, 53.3)
- moved R4 42.4 mm to (91.4, 58.4)
- moved R3 37.8 mm to (101.1, 67.3)
- moved J1 37.7 mm to (110.5, 39.4), turned to 90 degrees
- moved R5 37.4 mm to (96.0, 58.4)
- moved X1 36.0 mm to (111.8, 68.6)
- moved J2 34.6 mm to (94.0, 58.4)
- moved R2 26.2 mm to (95.2, 73.7)
- moved RV2 25.1 mm to (80.0, 82.5), turned to 90 degrees
- moved U1 23.8 mm to (110.5, 58.4)
- moved D1 22.1 mm to (102.9, 74.9)
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Other:
- board size 6.6 x 15.2 mm -> 15.2 x 6.7 mm
